File: RCJ2025_Board.kicad_sch (KiCad schematic)
At the start: 36 parts, among them J1 DCMotor1, J10 MicroGearedMotor, J11 Spare, J12 RSP_RESET, J2 DCMotor2, J3 TCS34725, J4 Encoder1, J5 Encoder1, J6 Encoder1, J7 Encoder1, J8 MotorBattery, J9 Servo, SW1 SW_DPDT_x2, U1 Pico

Commit message: ほぼ完成。最終確認待ち
Connections:
- net GND_RSP is gone; now on net GND: J12.2 (Pin_2), SW1.1 (A)
Changed lines of the file:
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@@
 	(paper "A4")
+	(junction
+		(at 101.6 80.01)
+		(diameter 0)
+		(color 0 0 0 0)
+	)
 	(junction
 		(at 58.42 132.08)
@@
 	)
 	(junction
+		(at 101.6 95.25)
+		(diameter 0)
+		(color 0 0 0 0)
+	)
+	(junction
 		(at 24.13 132.08)
 		(diameter 0)
@@
 	(wire
 		(pts
+			(xy 101.6 80.01) (xy 99.06 80.01)
+		)
+		(stroke
+			(width 0)
+			(type default)
+		)
+	)
+	(wire
+		(pts
 			(xy 58.42 151.13) (xy 58.42 156.21)
 		)
@@
 	(wire
 		(pts
+			(xy 104.14 95.25) (xy 101.6 95.25)
+		)
+		(stroke
+			(width 0)
+			(type default)
+		)
+	)
+	(wire
+		(pts
 			(xy 92.71 151.13) (xy 92.71 156.21)
 		)
@@
 	(wire
 		(pts
+			(xy 104.14 80.01) (xy 101.6 80.01)
+		)
+		(stroke
+			(width 0)
+			(type default)
+		)
+	)
+	(wire
+		(pts
 			(xy 49.53 146.05) (xy 49.53 151.13)
 		)
@@
 	(wire
 		(pts
+			(xy 101.6 80.01) (xy 101.6 95.25)
+		)
+		(stroke
+			(width 0)
+			(type default)
+		)
+	)
+	(wire
+		(pts
 			(xy 199.39 120.65) (xy 199.39 132.08)
 		)
@@
 	(wire
 		(pts
+			(xy 101.6 95.25) (xy 99.06 95.25)
+		)
+		(stroke
+			(width 0)
+			(type default)
+		)
+	)
+	(wire
+		(pts
 			(xy 100.33 120.65) (xy 100.33 132.08)
 		)
@@
 	(global_label "GND_RSP"
 		(shape input)
-		(at 99.06 80.01 0)
-		(fields_autoplaced yes)
-		(effects
-			(font
-				(size 1.27 1.27)
-			)
-			(justify left)
-		)
-		(property "Intersheetrefs" "${INTERSHEET_REFS}"
-			(at 110.6328 80.01 0)
+		(at 104.14 80.01 0)
+		(fields_autoplaced yes)
+		(effects
+			(font
+				(size 1.27 1.27)
+			)
+			(justify left)
+		)
+		(property "Intersheetrefs" "${INTERSHEET_REFS}"
+			(at 115.7128 80.01 0)
 			(effects
 				(font
@@
 	(global_label "GND"
 		(shape input)
-		(at 99.06 95.25 0)
-		(fields_autoplaced yes)
-		(effects
-			(font
-				(size 1.27 1.27)
-			)
-			(justify left)
-		)
-		(property "Intersheetrefs" "${INTERSHEET_REFS}"
-			(at 105.9157 95.25 0)
-			(effects
-				(font
+		(at 104.14 95.25 0)
+		(fields_autoplaced yes)
+		(effects
+			(font
+				(size 1.27 1.27)
+			)
+			(justify left)
+		)
+		(property "Intersheetrefs" "${INTERSHEET_REFS}"
+			(at 110.9957 95.25 0)
+			(effects
+				(font
