File: RCJ2025_Board.kicad_pcb (KiCad board)
At the start: 2 copper layers, 100 x 60 mm, 40 parts, among them J1 DCMotor1, J10 MicroGearedMotor, J11 Spare, J12 RSP_RESET, J2 DCMotor2, J3 TCS34725, J4 Encoder1, J5 Encoder1, J6 Encoder1, J7 Encoder1, J8 MotorBattery, J9 Servo, SW1 SW_DPDT_x2, U1 Pico

Commit message: 完成間際の絶望的状況
Parts:
- moved J12 77.7 mm to (187.5, 84.0), turned to 90 degrees
- moved SW1 71.0 mm to (187.5, 69.9)
- moved J11 59.0 mm to (159.5, 100.5)
- moved J7 47.5 mm to (163.5, 113.9)
- moved J6 46.8 mm to (159.5, 113.9)
- moved J5 45.3 mm to (155.5, 113.9)
- moved J3 44.7 mm to (146.5, 113.9)
- moved J4 44.7 mm to (151.5, 113.9)
- moved J1 40.1 mm to (105.0, 83.3), turned to 0 degrees
- moved BZ1 38.3 mm to (168.5, 102.0), turned to 90 degrees
- moved J8 31.5 mm to (181.0, 123.5)
- moved C4 30.9 mm to (181.0, 75.0), turned to 90 degrees
- moved C3 25.9 mm to (177.0, 75.0), turned to 90 degrees
- moved C8 24.1 mm to (181.0, 80.5), turned to 90 degrees
- moved J9 22.1 mm to (167.5, 113.9)
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Routing:
- net GND: track 0.00 -> 186.6 mm, vias 0 -> 300
- net 5V: track 0.00 -> 149.0 mm
- net 3.3V: track 0.00 -> 107.2 mm
- net Servo: track 0.00 -> 79.6 mm, vias 0 -> 1
- net RUN: track 0.00 -> 72.0 mm, vias 0 -> 2
- net B5: track 0.00 -> 71.9 mm
- net A5: track 0.00 -> 71.9 mm
- net 6V: track 0.00 -> 68.6 mm
- net SDA: track 0.00 -> 63.3 mm, vias 0 -> 2
- net SCL: track 0.00 -> 59.4 mm
- net GND_RSP: track 0.00 -> 50.2 mm, vias 0 -> 461
- net A2: track 0.00 -> 46.8 mm
- net A1: track 0.00 -> 46.2 mm
- net B2: track 0.00 -> 44.3 mm
- net B1: track 0.00 -> 43.7 mm
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Other:
- board text added: "${REFERENCE}"

Commit message: ほぼ完成。最終確認待ち
Parts:
- Raspberry Pi Pico: renamed from U1
- renumbered BNO1 to BNO055, BZ1 to Buzzer, J1 to DCMotor1, J2 to DCMotor2, J4 to Enc, J7 to Enc, J6 to Enc, J5 to Enc, J10 to MicroGearedMotor, J8 to MotorBattery, J12 to RSP_RST, J9 to Servo, J11 to Spare, J3 to TCS
Connections:
- RSP_RST pad 2: GND_RSP -> GND
- SW1 pad 1: GND_RSP -> GND
Routing:
- net GND_RSP: track 50.2 -> 0.00 mm, vias 461 -> 0
- net Servo: track 79.6 -> 82.3 mm
- net SDA: track 63.3 -> 65.3 mm
- net A5: track 71.9 -> 73.9 mm
- net SCL: track 59.4 -> 60.8 mm
- net 3.3V: track 107.2 -> 108.3 mm
- net 6V: track 68.6 -> 69.6 mm
- net GND: track 186.6 -> 187.5 mm, vias 300 -> 740
- net Buzzer: track 42.3 -> 43.2 mm
- net PWM2_A: track 20.7 -> 21.6 mm
- removed copper zone on B.Cu, net GND_RSP
- removed copper zone on F.Cu, net GND_RSP
Other:
- board text removed: "${REFERENCE}"

Commit message: ロゴマークを追加
Parts:
- added G***: LOGO, My_footprint:Remember_Logo, F.Cu at (172.0, 93.5)
- moved Buzzer 2.54 mm to (168.5, 104.5)
Routing:
- net Buzzer: track 43.2 -> 44.2 mm
- net GND: vias 740 -> 726
